Commit message: first real experiment tita controller

File: tita_controller/tita_description/tita.urdf (robot description, URDF)
Before this commit: robot tita, 15 links, 14 joints
Links:
- link left_leg_4: geometry collision cylinder length=0.034 radius=0.0925; visual mesh filename=meshes/left_leg_4.STL
- link right_leg_4: geometry collision cylinder length=0.034 radius=0.0925; visual mesh filename=meshes/right_leg_4.STL
